File: pcb/AC97.sch (KiCad schematic (older format))
At the start: 41 parts, among them J301 JACK_TRRS_6PINS, P301 RCA_2, P302 RCA_2, U301 LM4550, X301 24MHz

Commit message: ...
Parts:
- C301: value C -> 2.2u
- C310: value C -> 10u
- R301: value R -> 2.2K
- R302: value 1M -> 976K
- R307: value R -> 10K
- R317: value R -> 470
Changed lines of the file:
@@
 P 1850 1800
 F 0 "R302" V 1930 1800 50  0000 C CNN
-F 1 "1M" V 1850 1800 50  0000 C CNN
+F 1 "976K" V 1850 1800 50  0000 C CNN
 F 2 "Resistors_SMD:R_0805" V 1780 1800 50  0001 C CNN
 F 3 "" H 1850 1800 50  0000 C CNN
@@
 P 1200 6450
 F 0 "R301" V 1280 6450 50  0000 C CNN
-F 1 "R" V 1200 6450 50  0000 C CNN
+F 1 "2.2K" V 1200 6450 50  0000 C CNN
 F 2 "Resistors_SMD:R_0805" V 1130 6450 50  0001 C CNN
 F 3 "" H 1200 6450 50  0000 C CNN
@@
 P 1450 6700
 F 0 "C301" H 1475 6800 50  0000 L CNN
-F 1 "C" H 1475 6600 50  0000 L CNN
+F 1 "2.2u" H 1475 6600 50  0000 L CNN
 F 2 "Capacitors_SMD:C_0805" H 1488 6550 50  0001 C CNN
 F 3 "" H 1450 6700 50  0000 C CNN
@@
 P 1950 4200
 F 0 "R307" V 2030 4200 50  0000 C CNN
-F 1 "R" V 1950 4200 50  0000 C CNN
+F 1 "10K" V 1950 4200 50  0000 C CNN
 F 2 "Resistors_SMD:R_0805" V 1880 4200 50  0001 C CNN
 F 3 "" H 1950 4200 50  0000 C CNN
@@
 P 8600 6050
 F 0 "C310" H 8625 6150 50  0000 L CNN
-F 1 "C" H 8625 5950 50  0000 L CNN
+F 1 "10u" H 8625 5950 50  0000 L CNN
 F 2 "Capacitors_SMD:C_0805" H 8638 5900 50  0001 C CNN
 F 3 "" H 8600 6050 50  0001 C CNN
@@
 P 8900 5800
 F 0 "R317" V 8980 5800 50  0000 C CNN
-F 1 "R" V 8900 5800 50  0000 C CNN
+F 1 "470" V 8900 5800 50  0000 C CNN
 F 2 "Resistors_SMD:R_0805" V 8830 5800 50  0001 C CNN
 F 3 "" H 8900 5800 50  0001 C CNN
