File: pcb/AC97.sch (KiCad schematic (older format))
At the start: 37 parts, among them J301 JACK_TRRS_6PINS, P301 RCA_2, P302 RCA_2, U301 LM4550, X301 24MHz

Commit message: added schematic
Parts:
- added C318, C319, C320: 2.2u, Capacitors_SMD:C_0805, symbol C
- added R316: 10k, Resistors_SMD:R_0805, symbol R
- added unit 2 of U301
Connections:
- net +3V3: now also C319.1, U301.1 (DVDD), U301.9 (DVDD)
- net GND: now also C318.2, C319.2, C320.2, U301.26 (AVSS), U301.4 (DVSS), U301.7 (DVSS)
- net at C305.2, R302.1, U301.2 (XTL_IN): now also X301.1; no longer X301.3
- net at C302.2, R302.2, U301.3 (XTL_OUT): now also X301.3; no longer X301.1
- new net: C318.1, R316.2, U301.27 (VREF)
- new net +5V: C320.1, R316.1, U301.25 (AVDD)

Commit message: replaced ceramic DC blocking caps with electrolytics
Parts:
- removed C306, C307, C311: 47u, Capacitors_SMD:C_1206, symbol C
- added C306, C307: CP, Capacitors_ThroughHole:CP_Radial_D6.3mm_P2.50mm, symbol CP
- added R317: R, Resistors_SMD:R_0805, symbol R
- C310: value 47u -> C; footprint Capacitors_SMD:C_1206 -> Capacitors_SMD:C_0805
Connections:
- net +3V3: no longer R301.1
- net GND: now also C310.2
- net phone_l_out: now also C306.1
- net phone_left: now also C306.2
- net phone_r_out: now also C307.1; no longer C310.1
- net phone_right: now also C307.2; no longer C310.2
- net at U301.28 (VREF_OUT): now also R317.1
- new net mic_bias: C310.1, R301.1, R317.2

Commit message: fixed bad schematic symbols due to new kicad version
Parts:
- C301, C302, C303, C304, C305, C308, C309, C310, C312, C313, C314, C315, C316, C317, C318, C319, C320: symbol C -> ac97_pmod-rescue:C-RESCUE-ac97_pmod
- C306, C307: symbol CP -> ac97_pmod-rescue:CP-RESCUE-ac97_pmod
- J301: symbol JACK_TRRS_6PINS -> ac97_pmod-rescue:JACK_TRRS_6PINS-RESCUE-ac97_pmod
- P301, P302: symbol RCA_2 -> ac97_pmod-rescue:RCA_2-RESCUE-ac97_pmod
- R301, R302, R303, R304, R305, R306, R307, R308, R309, R310, R311, R312, R313, R314, R315, R316, R317: symbol R -> ac97_pmod-rescue:R-RESCUE-ac97_pmod
- U301: symbol LM4550 -> ac97_pmod-rescue:LM4550-RESCUE-ac97_pmod
- X301: symbol CRYSTAL_SMD_4 -> ac97_pmod-rescue:CRYSTAL_SMD_4-RESCUE-ac97_pmod

Commit message: updated symbol table
Parts:
- C310: value C -> 10u
- R301: value R -> 2.2K
- R302: value 1M -> 976K
- R307: value R -> 100K
- R317: value R -> 470
Changed lines of the file:
@@
 P 1850 1800
 F 0 "R302" V 1930 1800 50  0000 C CNN
-F 1 "1M" V 1850 1800 50  0000 C CNN
+F 1 "976K" V 1850 1800 50  0000 C CNN
 F 2 "Resistors_SMD:R_0805" V 1780 1800 50  0001 C CNN
 F 3 "" H 1850 1800 50  0000 C CNN
@@
 P 1200 6450
 F 0 "R301" V 1280 6450 50  0000 C CNN
-F 1 "R" V 1200 6450 50  0000 C CNN
+F 1 "2.2K" V 1200 6450 50  0000 C CNN
 F 2 "Resistors_SMD:R_0805" V 1130 6450 50  0001 C CNN
 F 3 "" H 1200 6450 50  0000 C CNN
@@
 P 1950 4200
 F 0 "R307" V 2030 4200 50  0000 C CNN
-F 1 "R" V 1950 4200 50  0000 C CNN
+F 1 "100K" V 1950 4200 50  0000 C CNN
 F 2 "Resistors_SMD:R_0805" V 1880 4200 50  0001 C CNN
 F 3 "" H 1950 4200 50  0000 C CNN
@@
 P 8600 6050
 F 0 "C310" H 8625 6150 50  0000 L CNN
-F 1 "C" H 8625 5950 50  0000 L CNN
+F 1 "10u" H 8625 5950 50  0000 L CNN
 F 2 "Capacitors_SMD:C_0805" H 8638 5900 50  0001 C CNN
 F 3 "" H 8600 6050 50  0001 C CNN
@@
 P 8900 5800
 F 0 "R317" V 8980 5800 50  0000 C CNN
-F 1 "R" V 8900 5800 50  0000 C CNN
+F 1 "470" V 8900 5800 50  0000 C CNN
 F 2 "Resistors_SMD:R_0805" V 8830 5800 50  0001 C CNN
 F 3 "" H 8900 5800 50  0001 C CNN
