File: pcb/PMOD_conn.sch (KiCad schematic (older format))
At the start: 3 parts, among them P401 CONN_02X06

Commit message: added schematic
Parts:
- P401: footprint Pin_Headers:Pin_Header_Angled_2x06 -> Pin_Headers:Pin_Header_Straight_2x06
Changed lines of the file:
@@
 F 0 "P401" H 3150 3000 50  0000 C CNN
 F 1 "CONN_02X06" H 3150 2300 50  0000 C CNN
-F 2 "Pin_Headers:Pin_Header_Angled_2x06" H 3150 1450 50  0001 C CNN
+F 2 "Pin_Headers:Pin_Header_Straight_2x06" H 3150 1450 50  0001 C CNN
 F 3 "" H 3150 1450 50  0000 C CNN
 	1    3150 2650
@@
 $EndComp
 $Comp
-L GND #PWR029
+L GND #PWR402
 U 1 1 577ED8FB
 P 3800 2800
-F 0 "#PWR029" H 3800 2550 50  0001 C CNN
+F 0 "#PWR402" H 3800 2550 50  0001 C CNN
 F 1 "GND" H 3800 2650 50  0000 C CNN
 F 2 "" H 3800 2800 50  0000 C CNN
@@
 $EndComp
 $Comp
-L GND #PWR030
+L GND #PWR401
 U 1 1 577ED912
 P 2500 2800
-F 0 "#PWR030" H 2500 2550 50  0001 C CNN
+F 0 "#PWR401" H 2500 2550 50  0001 C CNN
 F 1 "GND" H 2500 2650 50  0000 C CNN
 F 2 "" H 2500 2800 50  0000 C CNN
@@
 $EndComp
 $Comp
-L +3V3 #PWR031
+L +3V3 #PWR403
 U 1 1 577EDF28
 P 5700 1800
-F 0 "#PWR031" H 5700 1650 50  0001 C CNN
+F 0 "#PWR403" H 5700 1650 50  0001 C CNN
 F 1 "+3V3" H 5700 1940 50  0000 C CNN
 F 2 "" H 5700 1800 50  0000 C CNN
@@
 $EndComp
 $Comp
-L GND #PWR032
+L GND #PWR404
 U 1 1 577EDF45
 P 5700 2500
-F 0 "#PWR032" H 5700 2250 50  0001 C CNN
+F 0 "#PWR404" H 5700 2250 50  0001 C CNN
 F 1 "GND" H 5700 2350 50  0000 C CNN
 F 2 "" H 5700 2500 50  0000 C CNN

Commit message: fixed bad schematic symbols due to new kicad version
Parts:
- C401: symbol C -> ac97_pmod-rescue:C-RESCUE-ac97_pmod
- FB401: symbol FILTER -> ac97_pmod-rescue:FILTER-RESCUE-ac97_pmod
- P401: symbol CONN_02X06 -> ac97_pmod-rescue:CONN_02X06-RESCUE-ac97_pmod
Changed lines of the file:
@@
-EESchema Schematic File Version 3
-LIBS:power
-LIBS:device
-LIBS:transistors
-LIBS:conn
-LIBS:linear
-LIBS:regul
-LIBS:74xx
-LIBS:cmos4000
-LIBS:adc-dac
-LIBS:memory
-LIBS:xilinx
-LIBS:microcontrollers
-LIBS:dsp
-LIBS:microchip
-LIBS:analog_switches
-LIBS:motorola
-LIBS:texas
-LIBS:intel
-LIBS:audio
-LIBS:interface
-LIBS:digital-audio
-LIBS:philips
-LIBS:display
-LIBS:cypress
-LIBS:siliconi
-LIBS:opto
-LIBS:atmel
-LIBS:contrib
-LIBS:valves
-LIBS:wbraun_ic_lib
+EESchema Schematic File Version 4
 LIBS:ac97_pmod-cache
 EELAYER 26 0
@@
 $EndDescr
 $Comp
-L CONN_02X06 P401
+L ac97_pmod-rescue:CONN_02X06-RESCUE-ac97_pmod P401
 U 1 1 577ED8B8
 P 3150 2650
@@
 $EndComp
 $Comp
-L GND #PWR040
+L ac97_pmod-rescue:GND-RESCUE-ac97_pmod #PWR040
 U 1 1 577ED8FB
 P 3800 2800
@@
 $EndComp
 $Comp
-L GND #PWR041
+L ac97_pmod-rescue:GND-RESCUE-ac97_pmod #PWR041
 U 1 1 577ED912
 P 2500 2800
@@
 RESET
 $Comp
-L FILTER FB401
+L ac97_pmod-rescue:FILTER-RESCUE-ac97_pmod FB401
 U 1 1 577EDEB0
 P 5250 1900
@@
 $EndComp
 $Comp
-L C C401
+L ac97_pmod-rescue:C-RESCUE-ac97_pmod C401
 U 1 1 577EDEF4
 P 5700 2250
@@
 $EndComp
 $Comp
-L +3V3 #PWR042
+L ac97_pmod-rescue:+3V3-RESCUE-ac97_pmod #PWR042
 U 1 1 577EDF28
 P 5700 1800
@@
 $EndComp
 $Comp
-L GND #PWR043
+L ac97_pmod-rescue:GND-RESCUE-ac97_pmod #PWR043
 U 1 1 577EDF45
 P 5700 2500

Commit message: ...
Parts:
- C401: value 4.7uF -> 2.2u
Changed lines of the file:
@@
 P 5700 2250
 F 0 "C401" H 5725 2350 50  0000 L CNN
-F 1 "4.7uF" H 5725 2150 50  0000 L CNN
+F 1 "2.2u" H 5725 2150 50  0000 L CNN
 F 2 "Capacitors_SMD:C_0805" H 5738 2100 50  0001 C CNN
 F 3 "" H 5700 2250 50  0000 C CNN
