File: pcb/power_supply.sch (KiCad schematic (older format))
At the start: 8 parts, among them U201 MCP1640-*/CHY

Commit message: replaced ceramic DC blocking caps with electrolytics
Parts:
- added C204, C205: CP, Capacitors_ThroughHole:CP_Radial_D6.3mm_P2.50mm, symbol CP
Connections:
- net +3V3: now also C204.1
- net +5V: now also C205.1
- net GND: now also C204.2, C205.2
Changed lines of the file:
@@
-EESchema Schematic File Version 2
+EESchema Schematic File Version 3
 LIBS:power
 LIBS:device
@@
 LIBS:wbraun_ic_lib
 LIBS:ac97_pmod-cache
-EELAYER 25 0
+EELAYER 26 0
 EELAYER END
 $Descr A4 11693 8268
@@
 $EndComp
 $Comp
-L GND #PWR203
+L GND #PWR01
 U 1 1 576F6853
 P 2500 2600
-F 0 "#PWR203" H 2500 2350 50  0001 C CNN
+F 0 "#PWR01" H 2500 2350 50  0001 C CNN
 F 1 "GND" H 2500 2450 50  0000 C CNN
 F 2 "" H 2500 2600 50  0000 C CNN
@@
 $EndComp
 $Comp
-L GND #PWR204
+L GND #PWR02
 U 1 1 576F6879
 P 3900 3200
-F 0 "#PWR204" H 3900 2950 50  0001 C CNN
+F 0 "#PWR02" H 3900 2950 50  0001 C CNN
 F 1 "GND" H 3900 3050 50  0000 C CNN
 F 2 "" H 3900 3200 50  0000 C CNN
@@
 $EndComp
 $Comp
-L GND #PWR205
+L GND #PWR03
 U 1 1 576F689F
 P 4200 2800
-F 0 "#PWR205" H 4200 2550 50  0001 C CNN
+F 0 "#PWR03" H 4200 2550 50  0001 C CNN
 F 1 "GND" H 4200 2650 50  0000 C CNN
 F 2 "" H 4200 2800 50  0000 C CNN
@@
 $EndComp
 $Comp
-L GND #PWR202
+L GND #PWR04
 U 1 1 576F68E1
 P 2000 2700
-F 0 "#PWR202" H 2000 2450 50  0001 C CNN
+F 0 "#PWR04" H 2000 2450 50  0001 C CNN
 F 1 "GND" H 2000 2550 50  0000 C CNN
 F 2 "" H 2000 2700 50  0000 C CNN
@@
 $EndComp
 Wire Wire Line
-	2000 2300 2600 2300
+	1650 2300 2600 2300
 Wire Wire Line
 	2500 2400 2600 2400
@@
 Connection ~ 2500 2300
 $Comp
-L +3V3 #PWR201
+L +3V3 #PWR05
 U 1 1 576F6945
 P 2000 2200
-F 0 "#PWR201" H 2000 2050 50  0001 C CNN
+F 0 "#PWR05" H 2000 2050 50  0001 C CNN
 F 1 "+3V3" H 2000 2340 50  0000 C CNN
 F 2 "" H 2000 2200 50  0000 C CNN
@@
 $EndComp
 $Comp
-L +5V #PWR206
+L +5V #PWR06
 U 1 1 576F696B
 P 5400 2300
-F 0 "#PWR206" H 5400 2150 50  0001 C CNN
+F 0 "#PWR06" H 5400 2150 50  0001 C CNN
 F 1 "+5V" H 5400 2440 50  0000 C CNN
 F 2 "" H 5400 2300 50  0000 C CNN
@@
 $EndComp
 $Comp
-L GND #PWR207
+L GND #PWR07
 U 1 1 577EE208
 P 5400 2900
-F 0 "#PWR207" H 5400 2650 50  0001 C CNN
+F 0 "#PWR07" H 5400 2650 50  0001 C CNN
 F 1 "GND" H 5400 2750 50  0000 C CNN
 F 2 "" H 5400 2900 50  0000 C CNN
@@
 Connection ~ 4200 2400
 Wire Wire Line
-	5200 2400 5400 2400
+	5200 2400 5750 2400
 Wire Wire Line
 	5400 2300 5400 2500
@@
 	5400 2800 5400 2900
 Connection ~ 5400 2400
+$Comp
+L CP C204
+U 1 1 59E25F02
+P 1650 2450
+F 0 "C204" H 1675 2550 50  0000 L CNN
+F 1 "CP" H 1675 2350 50  0000 L CNN
+F 2 "Capacitors_ThroughHole:CP_Radial_D6.3mm_P2.50mm" H 1688 2300 50  0001 C CNN
+F 3 "" H 1650 2450 50  0001 C CNN
+	1    1650 2450
+	1    0    0    -1
+$EndComp
+$Comp
+L CP C205
+U 1 1 59E260A8
+P 5750 2650
+F 0 "C205" H 5775 2750 50  0000 L CNN
+F 1 "CP" H 5775 2550 50  0000 L CNN
+F 2 "Capacitors_ThroughHole:CP_Radial_D6.3mm_P2.50mm" H 5788 2500 50  0001 C CNN
+F 3 "" H 5750 2650 50  0001 C CNN
+	1    5750 2650
+	1    0    0    -1
+$EndComp
+$Comp
+L GND #PWR08
+U 1 1 59E26137
+P 5750 2900
+F 0 "#PWR08" H 5750 2650 50  0001 C CNN
+F 1 "GND" H 5750 2750 50  0000 C CNN
+F 2 "" H 5750 2900 50  0001 C CNN
+F 3 "" H 5750 2900 50  0001 C CNN
+	1    5750 2900
+	1    0    0    -1
+$EndComp
+Wire Wire Line
+	5750 2400 5750 2500
+Wire Wire Line
+	5750 2800 5750 2900
+Connection ~ 2000 2300
+$Comp
+L GND #PWR09
+U 1 1 59E2623D
+P 1650 2700
+F 0 "#PWR09" H 1650 2450 50  0001 C CNN
+F 1 "GND" H 1650 2550 50  0000 C CNN
+F 2 "" H 1650 2700 50  0001 C CNN
+F 3 "" H 1650 2700 50  0001 C CNN
+	1    1650 2700
+	1    0    0    -1
+$EndComp
+Wire Wire Line
+	1650 2600 1650 2700
 $EndSCHEMATC

Commit message: fixed bad schematic symbols due to new kicad version
Parts:
- C201, C202, C203: symbol C -> ac97_pmod-rescue:C-RESCUE-ac97_pmod
- C204, C205: symbol CP -> ac97_pmod-rescue:CP-RESCUE-ac97_pmod
- FB201: symbol FILTER -> ac97_pmod-rescue:FILTER-RESCUE-ac97_pmod
- L201: symbol INDUCTOR_SMALL -> ac97_pmod-rescue:INDUCTOR_SMALL-RESCUE-ac97_pmod
- R201, R202: symbol R -> ac97_pmod-rescue:R-RESCUE-ac97_pmod
- U201: symbol MCP1640-*/CHY -> wbraun_lib:MCP1640
Changed lines of the file:
@@
-EESchema Schematic File Version 3
-LIBS:power
-LIBS:device
-LIBS:transistors
-LIBS:conn
-LIBS:linear
-LIBS:regul
-LIBS:74xx
-LIBS:cmos4000
-LIBS:adc-dac
-LIBS:memory
-LIBS:xilinx
-LIBS:microcontrollers
-LIBS:dsp
-LIBS:microchip
-LIBS:analog_switches
-LIBS:motorola
-LIBS:texas
-LIBS:intel
-LIBS:audio
-LIBS:interface
-LIBS:digital-audio
-LIBS:philips
-LIBS:display
-LIBS:cypress
-LIBS:siliconi
-LIBS:opto
-LIBS:atmel
-LIBS:contrib
-LIBS:valves
-LIBS:wbraun_ic_lib
+EESchema Schematic File Version 4
 LIBS:ac97_pmod-cache
 EELAYER 26 0
@@
 $EndDescr
 $Comp
-L MCP1640-*/CHY U201
+L wbraun_lib:MCP1640 U201
 U 1 1 576F65ED
 P 3050 2400
@@
 $EndComp
 $Comp
-L C C201
+L ac97_pmod-rescue:C-RESCUE-ac97_pmod C201
 U 1 1 576F669D
 P 2000 2450
@@
 $EndComp
 $Comp
-L INDUCTOR_SMALL L201
+L ac97_pmod-rescue:INDUCTOR_SMALL-RESCUE-ac97_pmod L201
 U 1 1 576F66DD
 P 3050 1900
@@
 $EndComp
 $Comp
-L R R201
+L ac97_pmod-rescue:R-RESCUE-ac97_pmod R201
 U 1 1 576F6712
 P 3900 2550
@@
 $EndComp
 $Comp
-L R R202
+L ac97_pmod-rescue:R-RESCUE-ac97_pmod R202
 U 1 1 576F6764
 P 3900 2950
@@
 $EndComp
 $Comp
-L C C202
+L ac97_pmod-rescue:C-RESCUE-ac97_pmod C202
 U 1 1 576F6793
 P 4200 2550
@@
 $EndComp
 $Comp
-L GND #PWR01
+L ac97_pmod-rescue:GND-RESCUE-ac97_pmod #PWR01
 U 1 1 576F6853
 P 2500 2600
@@
 $EndComp
 $Comp
-L GND #PWR02
+L ac97_pmod-rescue:GND-RESCUE-ac97_pmod #PWR02
 U 1 1 576F6879
 P 3900 3200
@@
 $EndComp
 $Comp
-L GND #PWR03
+L ac97_pmod-rescue:GND-RESCUE-ac97_pmod #PWR03
 U 1 1 576F689F
 P 4200 2800
@@
 $EndComp
 $Comp
-L GND #PWR04
+L ac97_pmod-rescue:GND-RESCUE-ac97_pmod #PWR04
 U 1 1 576F68E1
 P 2000 2700
@@
 Connection ~ 2500 2300
 $Comp
-L +3V3 #PWR05
+L ac97_pmod-rescue:+3V3-RESCUE-ac97_pmod #PWR05
 U 1 1 576F6945
 P 2000 2200
+AR Path="/576F6945" Ref="#PWR05"  Part="1"
+AR Path="/576B2442/576F6945" Ref="#PWR05"  Part="1"
 F 0 "#PWR05" H 2000 2050 50  0001 C CNN
 F 1 "+3V3" H 2000 2340 50  0000 C CNN
@@
 $EndComp
 $Comp
-L +5V #PWR06
+L ac97_pmod-rescue:+5V-RESCUE-ac97_pmod #PWR06
 U 1 1 576F696B
 P 5400 2300
@@
 	2500 2500 2500 2600
 $Comp
-L FILTER FB201
+L ac97_pmod-rescue:FILTER-RESCUE-ac97_pmod FB201
 U 1 1 577EE17B
 P 4850 2400
@@
 $EndComp
 $Comp
-L C C203
+L ac97_pmod-rescue:C-RESCUE-ac97_pmod C203
 U 1 1 577EE1B6
 P 5400 2650
@@
 $EndComp
 $Comp
-L GND #PWR07
+L ac97_pmod-rescue:GND-RESCUE-ac97_pmod #PWR07
 U 1 1 577EE208
 P 5400 2900
@@
 Connection ~ 5400 2400
 $Comp
-L CP C204
+L ac97_pmod-rescue:CP-RESCUE-ac97_pmod C204
 U 1 1 59E25F02
 P 1650 2450
@@
 $EndComp
 $Comp
-L CP C205
+L ac97_pmod-rescue:CP-RESCUE-ac97_pmod C205
 U 1 1 59E260A8
 P 5750 2650
@@
 $EndComp
 $Comp
-L GND #PWR08
+L ac97_pmod-rescue:GND-RESCUE-ac97_pmod #PWR08
 U 1 1 59E26137
 P 5750 2900
@@
 Connection ~ 2000 2300
 $Comp
-L GND #PWR09
+L ac97_pmod-rescue:GND-RESCUE-ac97_pmod #PWR09
 U 1 1 59E2623D
 P 1650 2700

Commit message: updated symbol table
Parts:
- U201: symbol wbraun_lib:MCP1640 -> ac97_pmod-rescue:MCP1640-RESCUE-ac97_pmod
Changed lines of the file:
@@
 $EndDescr
 $Comp
-L wbraun_lib:MCP1640 U201
+L ac97_pmod-rescue:MCP1640-RESCUE-ac97_pmod U201
 U 1 1 576F65ED
 P 3050 2400
